File: PCB/LCD_0.96ST7735/LCD_0.96ST7735/LCD_0.96ST7735.kicad_sch (KiCad schematic)
At the start: 4 parts

Commit message: update
Parts:
- added H5, H6, H7, H8: MountingHole, MountingHole:MountingHole_3.2mm_M3, symbol Mechanical:MountingHole
- added J1, J3: Conn_02x10_Odd_Even, Connector_PinHeader_2.54mm:PinHeader_2x10_P2.54mm_Vertical, symbol Connector_Generic:Conn_02x10_Odd_Even
- added J2, J4: Conn_01x08_Male, Connector_PinHeader_2.00mm:PinHeader_1x08_P2.00mm_Vertical, symbol Connector:Conn_01x08_Male
- H1, H2, H3, H4: footprint MountingHole:MountingHole_3.2mm_M3_DIN965_Pad -> MountingHole:MountingHole_3.2mm_M3_Pad_Via
Connections:
- new net +3V3: J1.19 (Pin_19), J1.20 (Pin_20), J2.1 (Pin_1), J3.1 (Pin_1), J3.2 (Pin_2), J4.1 (Pin_1)
- new net +5V: J1.1 (Pin_1), J1.2 (Pin_2), J3.19 (Pin_19), J3.20 (Pin_20)
- new net BL: J2.8 (Pin_8), J4.8 (Pin_8)
- new net CLK: J2.4 (Pin_4), J3.9 (Pin_9), J4.4 (Pin_4)
- new net CS: J1.12 (Pin_12), J2.5 (Pin_5), J4.5 (Pin_5)
- new net DC: J1.9 (Pin_9), J2.6 (Pin_6), J4.6 (Pin_6)
- new net DIN: J2.3 (Pin_3), J3.6 (Pin_6), J4.3 (Pin_3)
- new net EN: J1.3 (Pin_3)
- new net GND: J1.17 (Pin_17), J1.18 (Pin_18), J2.2 (Pin_2), J3.3 (Pin_3), J3.4 (Pin_4), J4.2 (Pin_2)
- new net IO0: J3.16 (Pin_16)
- new net IO12: J1.11 (Pin_11)
- new net IO13: J3.18 (Pin_18)
- new net IO15: J3.17 (Pin_17)
- new net IO16: J3.14 (Pin_14)
- new net IO17: J3.11 (Pin_11)
- new net IO19: J3.10 (Pin_10)
- new net IO2: J3.15 (Pin_15)
- new net IO21: J3.7 (Pin_7)
- new net IO25: J1.7 (Pin_7)
- new net IO26: J1.10 (Pin_10)
- new net IO32: J1.5 (Pin_5)
- new net IO33: J1.8 (Pin_8), J2.7 (Pin_7), J4.7 (Pin_7)
- new net IO34: J1.4 (Pin_4)
- new net IO35: J1.6 (Pin_6)
- new net IO4: J3.13 (Pin_13)
- new net IO5: J3.12 (Pin_12)
- new net RXD0: J3.8 (Pin_8)
- new net TXD0: J3.5 (Pin_5)
- no-connect marks 0 -> 4
Other:
- moved on the sheet: H1, H2, H3, H4
