File: PCB/LCD_0.96ST7735/LCD_0.96ST7735/LCD_0.96ST7735.kicad_pcb (KiCad board)
At the start: 6 copper layers, 40 x 40 mm, 21 parts, among them J1 Conn_02x10_Odd_Even, J2 Conn_01x08_Male, J3 Conn_02x10_Odd_Even, J4 Conn_01x08_Male

Commit message: LCD_0.96_v1.1
Parts:
- removed kibuzzard-6404909D: G***, kibuzzard-6404909D
- added kibuzzard-64147912: G***, kibuzzard-64147912, B.Cu at (77.0, 119.1)
- J1, J3: moved to F.Cu
- moved J3 2.54 mm to (91.0, 90.8), turned to 0 degrees
- moved J1 2.54 mm to (60.5, 90.8), turned to 0 degrees
Routing:
- net /DC: track 54.4 -> 59.5 mm
- net /CLK: track 10.9 -> 7.41 mm
- net /DIN: track 8.68 -> 11.2 mm
- net GND: track 1.87 -> 0.00 mm
- net +3V3: track 1.87 -> 0.00 mm
- net /IO33: track 55.6 -> 56.4 mm
- net /CS: track 57.9 -> 58.7 mm
Other:
- board text added: "JLCJLCJLCJLC"
